File: eCAD/CAN_Bus.brd (EAGLE design)
At the start: 238.4 x 15.2 mm, 8 parts

Commit message: Rerouted CAN wires so that wires are of equivalent length
Routing:
- net CAN_L: track 237.3 -> 242.2 mm
- net 5V: track 200.3 -> 196.5 mm
