File: eCAD/Logging Board/Logging_board.brd (EAGLE design)
At the start: 72.1 x 45.7 mm, 16 parts, among them J3 SD_CARD_SOCKET

Commit message: Rev2 sent out for manufacturing.  Added 12MHz oscillator.  TODO: Add sign-of-life LED
Parts:
- added C2, C3: 18pF, SparkFun-Capacitors:CAP-PTH-2.54
- added Y1: 12MHz, SparkFun-Clocks:HC49US
- moved J2 6.84 mm to (58.4, 35.6)
- moved D1 4.58 mm to (21.6, 38.1), turned to 270 degrees
- moved D2 4.02 mm to (15.2, 38.1), turned to 270 degrees
- moved C1 3.81 mm to (43.2, 39.4), turned to 90 degrees
- moved D3 3.81 mm to (30.5, 41.9)
Connections:
- new net XTALIN: C2.2, LPC11C24.6, Y1.1
- new net XTALOUT: C3.2, LPC11C24.7, Y1.2
- net GND: now also C2.1, C3.1
Routing:
- net XTALIN: track 0.00 -> 40.4 mm
- net XTALOUT: track 0.00 -> 31.6 mm
- net V_SYS: track 68.7 -> 78.4 mm
- net GND: track 208.6 -> 202.1 mm, vias 0 -> 2
- net CAN_5V: track 25.8 -> 22.9 mm
- net N$1: track 27.1 -> 29.6 mm
Other:
- board text added: "Robobuggy Logging Board Rev 2"
- board text removed: "Robobuggy Logging Board Rev 1"

Commit message: Added missing sign-of-life LED and attached Vcc (CAN tranceiver power) to 5V bus
Parts:
- removed R4: 100, SparkFun-Resistors:AXIAL-0.3
- removed R5: 100k, SparkFun-Resistors:AXIAL-0.3
- removed RESET_SW: (no value), SparkFun-Switches:TACTILE_SWITCH_PTH_6.0MM
- added C8: 100nF, SparkFun-Capacitors:CAP-PTH-2.54
- added D4: GREEN, SparkFun-LED:LED-1206
- added R7: 100k, SparkFun-Resistors:AXIAL-0.3
- added R8: 13.6K, SparkFun-Resistors:AXIAL-0.3
- added R9: 100, SparkFun-Resistors:AXIAL-0.3
- added RESET_SW1: (no value), SparkFun-Switches:TACTILE_SWITCH_PTH_6.0MM
Connections:
- removed net N$2: R4.P$2, RESET_SW.1
- removed net VCC: LPC11C24.20
- new net N$5: D4.C, R8.P$2
- new net N$6: R9.P$2, RESET_SW1.3
- net CAN_5V: now also D4.A, LPC11C24.20, R7.P$2
- net GND: now also C8.2, LPC11C24.22, RESET_SW1.1; no longer R4.P$1
- net RESET: now also C8.1, R7.P$1, R8.P$1, R9.P$1; no longer R5.P$1, RESET_SW.3
- net V_SYS: no longer R5.P$2
Routing:
- net CAN_5V: track 22.9 -> 108.7 mm
- net GND: track 202.1 -> 136.9 mm
- net RESET: track 34.0 -> 42.5 mm, vias 1 -> 2
- net N$2: track 6.82 -> 0.00 mm
- net N$6: track 0.00 -> 5.86 mm
- net N$5: track 0.00 -> 3.02 mm
Other:
- board text added: "Robobuggy Logging Board Rev 3"
- board text removed: "Robobuggy Logging Board Rev 2"
