File: eCAD/Logging Board/Logging_board.sch (EAGLE design)
At the start: 19 parts, among them J3 SD_CARD_SOCKET, Y1 12MHz

Commit message: Added missing sign-of-life LED and attached Vcc (CAN tranceiver power) to 5V bus
Parts:
- removed R4: 100, SparkFun-Resistors:100OHM-HORIZ-1/4W-1%
- removed R5: 100k, SparkFun-Resistors:100KOHM-HORIZ-1/4W-1%
- removed RESET_SW: MOMENTARY-SWITCH-SPST-PTH-6.0MM, SparkFun-Switches:MOMENTARY-SWITCH-SPST-PTH-6.0MM
- added C8: 100nF, SparkFun-Capacitors:22PF-PTH-2.54MM-200V-5%
- added D4: GREEN, SparkFun-LED:LED-GREEN1206
- added R7: 100k, SparkFun-Resistors:100KOHM-HORIZ-1/4W-1%
- added R8: 13.6K, SparkFun-Resistors:100KOHM-HORIZ-1/4W-1%
- added R9: 100, SparkFun-Resistors:100KOHM-HORIZ-1/4W-1%
- added RESET_SW1: MOMENTARY-SWITCH-SPST-PTH-6.0MM, SparkFun-Switches:MOMENTARY-SWITCH-SPST-PTH-6.0MM
Connections:
- removed net N$2: R4.2, RESET_SW.1
- new net N$5: D4.C, R8.2
- new net N$6: R9.2, RESET_SW1.2
- net CAN_5V: now also D4.A, LPC11C24.VCC, R7.2
- net GND: now also C8.2, LPC11C24.STB, RESET_SW1.1; no longer R4.1
- net RESET: now also C8.1, R7.1, R8.1, R9.1; no longer R5.1, RESET_SW.2
- net V_SYS: no longer R5.2
Changed lines of the file:
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@@
 <layer number="59" name="tCarbon" color="7" fill="1" visible="no" active="no"/>
 <layer number="60" name="bCarbon" color="7" fill="1" visible="no" active="no"/>
+<layer number="88" name="SimResults" color="9" fill="1" visible="yes" active="yes"/>
+<layer number="89" name="SimProbes" color="9" fill="1" visible="yes" active="yes"/>
 <layer number="90" name="Modules" color="5" fill="1" visible="yes" active="yes"/>
 <layer number="91" name="Nets" color="2" fill="1" visible="yes" active="yes"/>
@@
 <part name="GND5" library="SparkFun-PowerSymbols" library_urn="urn:adsk.eagle:library:530" deviceset="GND" device=""/>
 <part name="ISP_SW" library="SparkFun-Switches" library_urn="urn:adsk.eagle:library:535" deviceset="MOMENTARY-SWITCH-SPST" device="-PTH-6.0MM" package3d_urn="urn:adsk.eagle:package:40163/1" value=""/>
-<part name="RESET_SW" library="SparkFun-Switches" library_urn="urn:adsk.eagle:library:535" deviceset="MOMENTARY-SWITCH-SPST" device="-PTH-6.0MM" package3d_urn="urn:adsk.eagle:package:40163/1" value=""/>
 <part name="R3" library="SparkFun-Resistors" library_urn="urn:adsk.eagle:library:532" deviceset="100OHM" device="-HORIZ-1/4W-1%" package3d_urn="urn:adsk.eagle:package:39658/1" value="100"/>
-<part name="R4" library="SparkFun-Resistors" library_urn="urn:adsk.eagle:library:532" deviceset="100OHM" device="-HORIZ-1/4W-1%" package3d_urn="urn:adsk.eagle:package:39658/1" value="100"/>
-<part name="GND6" library="SparkFun-PowerSymbols" library_urn="urn:adsk.eagle:library:530" deviceset="GND" device=""/>
-<part name="R5" library="SparkFun-Resistors" library_urn="urn:adsk.eagle:library:532" deviceset="100KOHM" device="-HORIZ-1/4W-1%" package3d_urn="urn:adsk.eagle:package:39658/1" value="100k"/>
 <part name="R6" library="SparkFun-Resistors" library_urn="urn:adsk.eagle:library:532" deviceset="100KOHM" device="-HORIZ-1/4W-1%" package3d_urn="urn:adsk.eagle:package:39658/1" value="100k"/>
 <part name="GND7" library="SparkFun-PowerSymbols" library_urn="urn:adsk.eagle:library:530" deviceset="GND" device=""/>
@@
 <part name="C3" library="SparkFun-Capacitors" library_urn="urn:adsk.eagle:library:510" deviceset="22PF" device="-PTH-2.54MM-200V-5%" package3d_urn="urn:adsk.eagle:package:37435/1" value="18pF"/>
 <part name="GND8" library="SparkFun-PowerSymbols" library_urn="urn:adsk.eagle:library:530" deviceset="GND" device=""/>
+<part name="RESET_SW1" library="SparkFun-Switches" library_urn="urn:adsk.eagle:library:535" deviceset="MOMENTARY-SWITCH-SPST" device="-PTH-6.0MM" package3d_urn="urn:adsk.eagle:package:40163/1" value=""/>
+<part name="GND9" library="SparkFun-PowerSymbols" library_urn="urn:adsk.eagle:library:530" deviceset="GND" device=""/>
+<part name="R7" library="SparkFun-Resistors" library_urn="urn:adsk.eagle:library:532" deviceset="100KOHM" device="-HORIZ-1/4W-1%" package3d_urn="urn:adsk.eagle:package:39658/1" value="100k"/>
+<part name="D4" library="SparkFun-LED" library_urn="urn:adsk.eagle:library:529" deviceset="LED-GREEN" device="1206" package3d_urn="urn:adsk.eagle:package:39352/1" value="GREEN"/>
+<part name="R8" library="SparkFun-Resistors" library_urn="urn:adsk.eagle:library:532" deviceset="100KOHM" device="-HORIZ-1/4W-1%" package3d_urn="urn:adsk.eagle:package:39658/1" value="13.6K"/>
+<part name="R9" library="SparkFun-Resistors" library_urn="urn:adsk.eagle:library:532" deviceset="100KOHM" device="-HORIZ-1/4W-1%" package3d_urn="urn:adsk.eagle:package:39658/1" value="100"/>
+<part name="C8" library="SparkFun-Capacitors" library_urn="urn:adsk.eagle:library:510" deviceset="22PF" device="-PTH-2.54MM-200V-5%" package3d_urn="urn:adsk.eagle:package:37435/1" value="100nF"/>
+<part name="GND11" library="SparkFun-PowerSymbols" library_urn="urn:adsk.eagle:library:530" deviceset="GND" device=""/>
+<part name="GND6" library="SparkFun-PowerSymbols" library_urn="urn:adsk.eagle:library:530" deviceset="GND" device=""/>
 </parts>
 <sheets>
@@
 <instance part="GND5" gate="1" x="-58.42" y="96.52"/>
 <instance part="ISP_SW" gate="G$1" x="83.82" y="-63.5"/>
-<instance part="RESET_SW" gate="G$1" x="-17.78" y="-73.66"/>
 <instance part="R3" gate="G$1" x="101.6" y="-63.5"/>
-<instance part="R4" gate="G$1" x="-33.02" y="-73.66"/>
-<instance part="GND6" gate="1" x="-48.26" y="-78.74"/>
-<instance part="R5" gate="G$1" x="-7.62" y="-63.5" rot="R90"/>
 <instance part="R6" gate="G$1" x="119.38" y="-55.88" rot="R90"/>
 <instance part="GND7" gate="1" x="73.66" y="-71.12"/>
@@
 <instance part="C3" gate="G$1" x="10.16" y="27.94" rot="R180"/>
 <instance part="GND8" gate="1" x="5.08" y="20.32"/>
+<instance part="RESET_SW1" gate="G$1" x="-22.86" y="-86.36"/>
+<instance part="GND9" gate="1" x="-38.1" y="-91.44"/>
+<instance part="R7" gate="G$1" x="2.54" y="-76.2" rot="R90"/>
+<instance part="D4" gate="G$1" x="15.24" y="-60.96"/>
+<instance part="R8" gate="G$1" x="15.24" y="-76.2" rot="R90"/>
+<instance part="R9" gate="G$1" x="-7.62" y="-86.36" rot="R180"/>
+<instance part="C8" gate="G$1" x="-2.54" y="-91.44"/>
+<instance part="GND11" gate="1" x="-2.54" y="-96.52"/>
+<instance part="GND6" gate="1" x="93.98" y="-25.4"/>
 </instances>
 <busses>
@@
 <wire x1="-60.96" y1="99.06" x2="-58.42" y2="99.06" width="0.1524" layer="91"/>
 <pinref part="GND5" gate="1" pin="GND"/>
-</segment>
-<segment>
-<pinref part="R4" gate="G$1" pin="1"/>
-<wire x1="-38.1" y1="-73.66" x2="-48.26" y2="-73.66" width="0.1524" layer="91"/>
-<wire x1="-48.26" y1="-73.66" x2="-48.26" y2="-76.2" width="0.1524" layer="91"/>
-<pinref part="GND6" gate="1" pin="GND"/>
 </segment>
 <segment>
@@
 <junction x="5.08" y="22.86"/>
 </segment>
+<segment>
+<wire x1="-27.94" y1="-86.36" x2="-38.1" y2="-86.36" width="0.1524" layer="91"/>
+<wire x1="-38.1" y1="-86.36" x2="-38.1" y2="-88.9" width="0.1524" layer="91"/>
+<pinref part="GND9" gate="1" pin="GND"/>
+<pinref part="RESET_SW1" gate="G$1" pin="1"/>
+</segment>
+<segment>
+<pinref part="C8" gate="G$1" pin="2"/>
+<pinref part="GND11" gate="1" pin="GND"/>
+</segment>
+<segment>
+<pinref part="LPC11C24" gate="G$1" pin="STB"/>
+<pinref part="GND6" gate="1" pin="GND"/>
+</segment>
 </net>
 <net name="V_SYS" class="0">
@@
 <wire x1="38.1" y1="12.7" x2="27.94" y2="12.7" width="0.1524" layer="91"/>
 <label x="27.94" y="12.7" size="1.778" layer="95"/>
-</segment>
-<segment>
-<pinref part="R5" gate="G$1" pin="2"/>
-<wire x1="-7.62" y1="-58.42" x2="-7.62" y2="-55.88" width="0.1524" layer="91"/>
-<wire x1="-7.62" y1="-55.88" x2="-2.54" y2="-55.88" width="0.1524" layer="91"/>
-<label x="-5.08" y="-55.88" size="1.778" layer="95"/>
 </segment>
 <segment>
@@
 <pinref part="R2" gate="G$1" pin="1"/>
 </segment>
+<segment>
+<pinref part="LPC11C24" gate="G$1" pin="VCC"/>
+<wire x1="38.1" y1="7.62" x2="25.4" y2="7.62" width="0.1524" layer="91"/>
+<label x="25.4" y="7.62" size="1.778" layer="95"/>
+</segment>
+<segment>
+<pinref part="R7" gate="G$1" pin="2"/>
+<wire x1="2.54" y1="-71.12" x2="2.54" y2="-55.88" width="0.1524" layer="91"/>
+<wire x1="2.54" y1="-55.88" x2="15.24" y2="-55.88" width="0.1524" layer="91"/>
+<pinref part="D4" gate="G$1" pin="A"/>
+<wire x1="15.24" y1="-55.88" x2="25.4" y2="-55.88" width="0.1524" layer="91"/>
+<wire x1="15.24" y1="-58.42" x2="15.24" y2="-55.88" width="0.1524" layer="91"/>
+<junction x="15.24" y="-55.88"/>
+<label x="20.32" y="-55.88" size="1.778" layer="95"/>
+</segment>
 </net>
 <net name="CAN_H" class="0">
@@
 </segment>
 </net>
-<net name="N$2" class="0">
-<segment>
-<pinref part="R4" gate="G$1" pin="2"/>
-<pinref part="RESET_SW" gate="G$1" pin="1"/>
-<wire x1="-27.94" y1="-73.66" x2="-22.86" y2="-73.66" width="0.1524" layer="91"/>
-</segment>
-</net>
 <net name="RESET" class="0">
-<segment>
-<pinref part="RESET_SW" gate="G$1" pin="2"/>
-<wire x1="-12.7" y1="-73.66" x2="-7.62" y2="-73.66" width="0.1524" layer="91"/>
-<label x="0" y="-73.66" size="1.778" layer="95"/>
-<wire x1="-7.62" y1="-73.66" x2="2.54" y2="-73.66" width="0.1524" layer="91"/>
-<wire x1="-7.62" y1="-73.66" x2="-7.62" y2="-68.58" width="0.1524" layer="91"/>
-<junction x="-7.62" y="-73.66"/>
-<pinref part="R5" gate="G$1" pin="1"/>
-</segment>
 <segment>
 <pinref part="LPC11C24" gate="G$1" pin="!RESET!/PIO0_0"/>
 <wire x1="93.98" y1="88.9" x2="119.38" y2="88.9" width="0.1524" layer="91"/>
 <label x="109.22" y="88.9" size="1.778" layer="95"/>
+</segment>
+<segment>
+<label x="27.94" y="-86.36" size="1.778" layer="95"/>
+<wire x1="2.54" y1="-86.36" x2="2.54" y2="-81.28" width="0.1524" layer="91"/>
+<pinref part="R7" gate="G$1" pin="1"/>
+<wire x1="2.54" y1="-86.36" x2="15.24" y2="-86.36" width="0.1524" layer="91"/>
+<pinref part="R8" gate="G$1" pin="1"/>
+<wire x1="15.24" y1="-86.36" x2="27.94" y2="-86.36" width="0.1524" layer="91"/>
+<wire x1="15.24" y1="-81.28" x2="15.24" y2="-86.36" width="0.1524" layer="91"/>
+<junction x="15.24" y="-86.36"/>
+<pinref part="R9" gate="G$1" pin="1"/>
+<wire x1="2.54" y1="-86.36" x2="-2.54" y2="-86.36" width="0.1524" layer="91"/>
+<junction x="2.54" y="-86.36"/>
+<pinref part="C8" gate="G$1" pin="1"/>
+<junction x="-2.54" y="-86.36"/>
 </segment>
 </net>
@@
 </segment>
 </net>
+<net name="N$5" class="0">
+<segment>
+<pinref part="D4" gate="G$1" pin="C"/>
+<pinref part="R8" gate="G$1" pin="2"/>
+<wire x1="15.24" y1="-66.04" x2="15.24" y2="-71.12" width="0.1524" layer="91"/>
+</segment>
+</net>
+<net name="N$6" class="0">
+<segment>
+<pinref part="R9" gate="G$1" pin="2"/>
+<pinref part="RESET_SW1" gate="G$1" pin="2"/>
+<wire x1="-12.7" y1="-86.36" x2="-17.78" y2="-86.36" width="0.1524" layer="91"/>
+</segment>
+</net>
