File: eCAD/Steering Board/Steering Controller.sch (EAGLE design)
At the start: 22 parts, among them Y1 12MHz

Commit message: Added new pin headers & tri-state buffers
-New 3-pin header to communicate with NAND Servo
-Removed Obsolete 2pin header
-Updated DB9 and UART
-Added Tri-State Buffers to control TXD/RXD data flow.
Parts:
- removed J3: (no value), SparkFun-Connectors:CONN_04
- added R4, R7: 10k, SparkFun-Resistors:100KOHM-HORIZ-1/4W-1%
- added U1, U2, U3: SN74LVC2G241, AdamLibrary:SN74LVC2G241
- J4: device SparkFun-Connectors:CONN_02 -> SparkFun-Connectors:CONN_03
Connections:
- removed net ENC_A: J3.3, LPC11C24.PIO0_2/SSEL0/CT16B0_CAP0
- removed net ENC_B: J3.2, LPC11C24.PIO0_5/SDA
- removed net STEER_PWM: J4.1, LPC11C24.PIO0_8/MISO0/CT16B0_MAT0
- new net +12V: J1.5, J4.2
- new net DATA: J4.3, R4.1, U3.1IN, U3.2OUT
- new net N$3: U2.1IN, U3.1OUT
- new net N$5: U1.1OUT, U3.2IN
- new net TX_ENABLE: LPC11C24.PIO0_2/SSEL0/CT16B0_CAP0, U3.2OE, U3.~1OE
- new net UART_5V: J2.4, R7.2, U1.~1OE, U2.~1OE
- net 3.3V: now also R4.2, U1.VCC, U2.VCC, U3.VCC
- net CAN_5V: no longer J3.1
- net GND: now also J4.1, R7.1, U1.2IN, U1.2OE, U1.2OUT, U1.GND, U2.2IN, U2.2OE, U2.2OUT, U2.GND, U3.GND; no longer J3.4, J4.2
- net RXD: now also U2.1OUT
- net TXD: now also U1.1IN
